Commit message: Started adding ability for spawned Gazebo model to move with controllers

File: src/srr_sim/urdf/srr.urdf (robot description, URDF)
Before this commit: robot srr, 10 links, 9 joints
Joints:
- joint FL_Joint: limit lower=0 upper=0 effort=0 velocity=0 -> lower=0 upper=1.5707963 effort=0 velocity=0
- joint FR_Joint: limit lower=0 upper=0 effort=0 velocity=0 -> lower=0 upper=1.5707963 effort=0 velocity=0
- joint RL_Joint: limit lower=0 upper=0 effort=0 velocity=0 -> lower=0 upper=1.5707963 effort=0 velocity=0
- joint RR_Joint: limit lower=0 upper=0 effort=0 velocity=0 -> lower=0 upper=1.5707963 effort=0 velocity=0

File: src/srr_sim/urdf/srr_integrated.urdf.xacro (robot description, xacro)
@@ -2,4 +2,78 @@
 <robot name ="srr_integrated" xmlns:xacro="http://wiki.ros.org/xacro">
   <xacro:include filename="srr.urdf"/>
+  <!-- ROBOT JOINT TRANSMISSIONS -->
+  <transmission name="FR_Transmitter">
+    <type>transmission_interface/SimpleTransmission</type>
+    <joint name="FR_Joint">
+      <hardwareInterface>hardware_interface/EffortJointInterface</hardwareInterface>
+    </joint>
+    <actuator name="FR_Motor">
+      <mechanicalReduction>50</mechanicalReduction>
+    </actuator>
+  </transmission>
+  <transmission name="FL_Transmitter">
+    <type>transmission_interface/SimpleTransmission</type>
+    <joint name="FL_Joint">
+      <hardwareInterface>hardware_interface/EffortJointInterface</hardwareInterface>
+    </joint>
+    <actuator name="FL_Motor">
+      <mechanicalReduction>50</mechanicalReduction>
+    </actuator>
+  </transmission>
+  <transmission name="RR_Transmitter">
+    <type>transmission_interface/SimpleTransmission</type>
+    <joint name="RR_Joint">
+      <hardwareInterface>hardware_interface/EffortJointInterface</hardwareInterface>
+    </joint>
+    <actuator name="RR_Motor">
+      <mechanicalReduction>50</mechanicalReduction>
+    </actuator>
+  </transmission>
+  <transmission name="RL_Transmitter">
+    <type>transmission_interface/SimpleTransmission</type>
+    <joint name="RL_Joint">
+      <hardwareInterface>hardware_interface/EffortJointInterface</hardwareInterface>
+    </joint>
+    <actuator name="RL_Motor">
+      <mechanicalReduction>50</mechanicalReduction>
+    </actuator>
+  </transmission>
+  <transmission name="FR_Wheel_Transmitter">
+    <type>transmission_interface/SimpleTransmission</type>
+    <joint name="FR_Wheel_Joint">
+      <hardwareInterface>hardware_interface/EffortJointInterface</hardwareInterface>
+    </joint>
+    <actuator name="FR_Wheel_Motor">
+      <mechanicalReduction>50</mechanicalReduction>
+    </actuator>
+  </transmission>
+  <transmission name="FL_Wheel_Transmitter">
+    <type>transmission_interface/SimpleTransmission</type>
+    <joint name="FL_Wheel_Joint">
+      <hardwareInterface>hardware_interface/EffortJointInterface</hardwareInterface>
+    </joint>
+    <actuator name="FL_Wheel_Motor">
+      <mechanicalReduction>50</mechanicalReduction>
+    </actuator>
+  </transmission>
+  <transmission name="RR_Wheel_Transmitter">
+    <type>transmission_interface/SimpleTransmission</type>
+    <joint name="RR_Wheel_Joint">
+      <hardwareInterface>hardware_interface/EffortJointInterface</hardwareInterface>
+    </joint>
+    <actuator name="RR_Wheel_Motor">
+      <mechanicalReduction>50</mechanicalReduction>
+    </actuator>
+  </transmission>
+  <transmission name="RL_Wheel_Transmitter">
+    <type>transmission_interface/SimpleTransmission</type>
+    <joint name="RL_Wheel_Joint">
+      <hardwareInterface>hardware_interface/EffortJointInterface</hardwareInterface>
+    </joint>
+    <actuator name="RL_Wheel_Motor">
+      <mechanicalReduction>50</mechanicalReduction>
+    </actuator>
+  </transmission>
+  <!-- ROS CONTROL LIBRARY -->
   <gazebo>
     <plugin name="gazebo_ros_control" filename="libgazebo_ros_control.so">

Commit message: Added missing controller management node to launch file, standardized namespaces

File: src/srr_sim/urdf/srr.urdf (robot description, URDF)
Before this commit: robot srr, 10 links, 9 joints
Joints:
- joint FL_Joint: limit lower=0 upper=1.5707963 effort=0 velocity=0 -> lower=0 upper=1.5707963 effort=100 velocity=0
- joint FR_Joint: limit lower=0 upper=1.5707963 effort=0 velocity=0 -> lower=0 upper=1.5707963 effort=100 velocity=0
- joint RL_Joint: limit lower=0 upper=1.5707963 effort=0 velocity=0 -> lower=0 upper=1.5707963 effort=100 velocity=0
- joint RR_Joint: limit lower=0 upper=1.5707963 effort=0 velocity=0 -> lower=0 upper=1.5707963 effort=100 velocity=0

File: src/srr_sim/urdf/srr_integrated.urdf.xacro (robot description, xacro)
@@ -78,5 +78,5 @@
   <gazebo>
     <plugin name="gazebo_ros_control" filename="libgazebo_ros_control.so">
-      <robotNamespace>/srr</robotNamespace>
+      <robotNamespace>/srr_integrated</robotNamespace>
       <robotSimType>gazebo_ros_control/DefaultRobotHWSim</robotSimType>
       <legacyModeNS>true</legacyModeNS>

Commit message: Added initial srr_teleop package with minimally proven joint controller connections and dumb teleop script

File: src/srr_sim/urdf/srr.urdf (robot description, URDF)
Before this commit: robot srr, 10 links, 9 joints
Joints:
- joint FL_Joint: limit lower=0 upper=1.5707963 effort=100 velocity=0 -> lower=0 upper=1.5707963 effort=12.5 velocity=0
- joint FL_Wheel_Joint: limit (none) -> effort=12.5 velocity=0
- joint FR_Joint: limit lower=0 upper=1.5707963 effort=100 velocity=0 -> lower=0 upper=1.5707963 effort=12.5 velocity=0
- joint FR_Wheel_Joint: limit (none) -> effort=12.5 velocity=0
- joint RL_Joint: limit lower=0 upper=1.5707963 effort=100 velocity=0 -> lower=0 upper=1.5707963 effort=12.5 velocity=0
- joint RL_Wheel_Joint: limit (none) -> effort=12.5 velocity=0
- joint RR_Joint: limit lower=0 upper=1.5707963 effort=100 velocity=0 -> lower=0 upper=1.5707963 effort=12.5 velocity=0
- joint RR_Wheel_Joint: limit (none) -> effort=12.5 velocity=0

Commit message: Slightly adjusted joint effort limits (and reordered XML block)

File: src/srr_sim/urdf/srr.urdf (robot description, URDF)
Before this commit: robot srr, 10 links, 9 joints
Joints:
- joint FL_Joint: limit lower=0 upper=1.5707963 effort=12.5 velocity=0 -> lower=0 upper=1.5707963 effort=125 velocity=0
- joint FR_Joint: limit lower=0 upper=1.5707963 effort=12.5 velocity=0 -> lower=0 upper=1.5707963 effort=125 velocity=0
- joint RL_Joint: limit lower=0 upper=1.5707963 effort=12.5 velocity=0 -> lower=0 upper=1.5707963 effort=125 velocity=0
- joint RR_Joint: limit lower=0 upper=1.5707963 effort=12.5 velocity=0 -> lower=0 upper=1.5707963 effort=125 velocity=0

Commit message: Added vehicle chassis joint offsets to rosparam server, had force positions script account for offsets
Also opened up the joint position limits temporarily, just for testing and such.

File: src/srr_sim/urdf/srr.urdf (robot description, URDF)
Before this commit: robot srr, 10 links, 9 joints
Joints:
- joint FL_Joint: limit lower=0 upper=1.5707963 effort=125 velocity=0 -> lower=-1.5707963 upper=1.5707963 effort=125 velocity=0
- joint FR_Joint: limit lower=0 upper=1.5707963 effort=125 velocity=0 -> lower=-1.5707963 upper=1.5707963 effort=125 velocity=0
- joint RL_Joint: limit lower=0 upper=1.5707963 effort=125 velocity=0 -> lower=-1.5707963 upper=1.5707963 effort=125 velocity=0
- joint RR_Joint: limit lower=0 upper=1.5707963 effort=125 velocity=0 -> lower=-1.5707963 upper=1.5707963 effort=125 velocity=0

Commit message: Changed controllers to velocity controllers, tweaked teleop and URDF limits

File: src/srr_sim/urdf/srr.urdf (robot description, URDF)
Before this commit: robot srr, 14 links, 13 joints
Joints:
- joint FL_Joint: limit lower=-0.767945 upper=0.0 effort=125 velocity=0 -> lower=-0.767945 upper=0.0 effort=125 velocity=1.25
- joint FL_Rev_Joint: limit lower=-0.02 upper=0.02 effort=125 velocity=0 -> lower=-0.2618 upper=0.2618 effort=125 velocity=0
- joint FL_Wheel_Joint: limit effort=12.5 velocity=0 -> effort=12.5 velocity=2.5
- joint FR_Joint: limit lower=-0.767945 upper=0.0 effort=125 velocity=0 -> lower=-0.767945 upper=0.0 effort=125 velocity=1.25
- joint FR_Rev_Joint: limit lower=-0.02 upper=0.02 effort=125 velocity=0 -> lower=-0.2618 upper=0.2618 effort=125 velocity=0
- joint FR_Wheel_Joint: limit effort=12.5 velocity=0 -> effort=12.5 velocity=2.5
- joint RL_Joint: limit lower=0.0 upper=0.767945 effort=125 velocity=0 -> lower=0.0 upper=0.767945 effort=125 velocity=1.25
- joint RL_Wheel_Joint: limit effort=12.5 velocity=0 -> effort=12.5 velocity=2.5
- joint RR_Joint: limit lower=0.0 upper=0.767945 effort=125 velocity=0 -> lower=0.0 upper=0.767945 effort=125 velocity=1.25
- joint RR_Wheel_Joint: limit effort=12.5 velocity=0 -> effort=12.5 velocity=2.5

Commit message: Improved robot structure by adding the ability to steer the front wheels

File: src/srr_sim/urdf/srr.urdf (robot description, URDF)
Before this commit: robot srr, 10 links, 9 joints
Links:
- added link Front_Left_Rev_Link, mass 0.063238; collision mesh filename=package://srr_sim/meshes/Front_Left_Rev_Link.STL; visual mesh filename=package://srr_sim/meshes/Front_Left_Rev_Link.STL
- added link Front_Right_Rev_Link, mass 0.1436780324417; collision mesh filename=package://srr_sim/meshes/Front_Right_Rev_Link.STL; visual mesh filename=package://srr_sim/meshes/Front_Right_Rev_Link.STL
- link Front_Left: mass 0.13037 -> 0.097852
- link Front_Left_Wheel: mass 0.68474 -> 0.72193847666214
- link Front_Right: mass 0.13037 -> 0.0978518395980198
- link Front_Right_Wheel: mass 0.684735063470279 -> 0.72194
- link Rear_Left: mass 0.13037 -> 0.13036735305509
- link Rear_Left_Wheel: mass 0.684735063470277 -> 0.69177
- link Rear_Right_Wheel: mass 0.68474 -> 0.691773547047117
Joints:
- added joint FL_Rev_Joint: type revolute, parent Front_Left, child Front_Left_Rev_Link, origin xyz=0.21838 0.0052363 -0.01905 rpy=0 0.036515 0.023974, axis 0 1 0, limit lower=-0.218166 upper=0.218166 effort=125 velocity=0
- added joint FR_Rev_Joint: type revolute, parent Front_Right, child Front_Right_Rev_Link, origin xyz=0.21198 0.052735 0.01905 rpy=0 -0.0080108 0.24382, axis 0 1 0, limit lower=-0.218166 upper=0.218166 effort=125 velocity=0
- joint FL_Joint: origin xyz=0 0.15621 0.034606 rpy=1.5708 0.23089 0 -> xyz=0 0.15621 0.034606 rpy=1.5708 0 0
- joint FL_Wheel_Joint: origin xyz=0.25908 0 0 rpy=0 0 -0.79784 -> xyz=0 -0.06096 0 rpy=0 0 -0.75345; parent Front_Left -> Front_Left_Rev_Link
- joint FR_Joint: origin xyz=0 -0.15621 0.034606 rpy=1.5708 0.43239 0 -> xyz=0 -0.15621 0.034606 rpy=1.5708 0 0
- joint FR_Wheel_Joint: origin xyz=0.25908 0 0 rpy=0 0 -2.5083 -> xyz=0 -0.06096 0 rpy=0 0 -1.311; parent Front_Right -> Front_Right_Rev_Link
- joint RL_Joint: origin xyz=0 0.18161 0.034606 rpy=1.5708 -0.38556 0 -> xyz=0 0.18161 0.034606 rpy=1.5708 0 0
- joint RL_Wheel_Joint: origin xyz=-0.25908 0 0 rpy=0 0 -0.610274581412076 -> xyz=-0.25908 0 0 rpy=0 0 -0.61027
- joint RR_Joint: origin xyz=0 -0.18161 0.034606 rpy=1.5708 -0.37306 0 -> xyz=0 -0.18161 0.0346062035203441 rpy=1.5707963267949 0 0
- joint RR_Wheel_Joint: origin xyz=-0.25908 0 0 rpy=0 0 -0.397587942822765 -> xyz=-0.25908 0 0 rpy=0 0 -0.39759

Commit message: Mirrored new front leg structure to back legs as well
The same components that were added to the front legs were added to the
back, but there's no steering mechanism for the rear wheels, the fixed
joint keeps the wheels facing forward

File: src/srr_sim/urdf/srr.urdf (robot description, URDF)
Before this commit: robot srr, 12 links, 11 joints
Links:
- added link Rear_Left_Fixed_Link, mass 0.063238; collision mesh filename=package://srr_sim/meshes/Rear_Left_Fixed_Link.STL; visual mesh filename=package://srr_sim/meshes/Rear_Left_Fixed_Link.STL
- added link Rear_Right_Fixed_Link, mass 0.0632382201349725; collision mesh filename=package://srr_sim/meshes/Rear_Right_Fixed_Link.STL; visual mesh filename=package://srr_sim/meshes/Rear_Right_Fixed_Link.STL
- link Front_Left: mass 0.097852 -> 0.0978518500972839
- link Front_Left_Rev_Link: mass 0.063238 -> 0.0632382201349724
- link Front_Right: mass 0.0978518395980198 -> 0.0978518506132432
- link Front_Right_Rev_Link: mass 0.1436780324417 -> 0.0632382201349724
- link Front_Right_Wheel: mass 0.72194 -> 0.721938476662141
- link Rear_Left: mass 0.13036735305509 -> 0.097851850152702
- link Rear_Left_Wheel: mass 0.69177 -> 0.72193847666214
- link Rear_Right: mass 0.13036735305509 -> 0.0978518501695887
- link Rear_Right_Wheel: mass 0.691773547047117 -> 0.72194
- link base_link: mass 16.6773118924852 -> 16.6873668690236
Joints:
- added joint RL_Fixed_Joint: type fixed, parent Rear_Left, child Rear_Left_Fixed_Link, origin xyz=0.21844 0.01651 -0.022225 rpy=0 0 3.1416, axis 0 0 0
- added joint RR_Fixed_Joint: type fixed, parent Rear_Right, child Rear_Right_Fixed_Link, origin xyz=0.21844 0.01651 0.022225 rpy=0 0 3.1416, axis 0 0 0
- joint FL_Joint: origin xyz=0 0.15621 0.034606 rpy=1.5708 0 0 -> xyz=0 0.15304 0.034606 rpy=1.5708 0 0
- joint FL_Rev_Joint: origin xyz=0.21838 0.0052363 -0.01905 rpy=0 0.036515 0.023974 -> xyz=0.21844 0 -0.022225 rpy=0 -0.0077095 0
- joint FL_Wheel_Joint: origin xyz=0 -0.06096 0 rpy=0 0 -0.75345 -> xyz=0 -0.06096 0 rpy=0 0 -1.2844
- joint FR_Joint: origin xyz=0 -0.15621 0.034606 rpy=1.5708 0 0 -> xyz=0 -0.153035 0.0346062035203441 rpy=1.5707963267949 0 0
- joint FR_Rev_Joint: origin xyz=0.21198 0.052735 0.01905 rpy=0 -0.0080108 0.24382 -> xyz=0.21844 0 0.022225 rpy=0 0.031575 0
- joint FR_Wheel_Joint: origin xyz=0 -0.06096 0 rpy=0 0 -1.311 -> xyz=0 -0.06096 0 rpy=0 0 -1.2319
- joint RL_Joint: origin xyz=0 0.18161 0.034606 rpy=1.5708 0 0 -> xyz=0 0.17844 0.034606 rpy=-1.5708 0 -3.1416
- joint RL_Wheel_Joint: origin xyz=-0.25908 0 0 rpy=0 0 -0.61027 -> xyz=0 -0.04445 0 rpy=0 0 0.62124; parent Rear_Left -> Rear_Left_Fixed_Link
- joint RR_Joint: origin xyz=0 -0.18161 0.0346062035203441 rpy=1.5707963267949 0 0 -> xyz=0 -0.17844 0.034606 rpy=-1.5708 0 -3.1416
- joint RR_Wheel_Joint: origin xyz=-0.25908 0 0 rpy=0 0 -0.39759 -> xyz=0 -0.04445 0 rpy=0 0 3.0007; parent Rear_Right -> Rear_Right_Fixed_Link

Commit message: Added the elements to sim the basic arm (URDF, STL, etc)
Also moved the srr STL files to new srr subdirectory and put sample return arm
(sra) to its own sra subdirectory. Created launch file that mounts the arm to
the world's origin frame.

File: src/srr_sim/urdf/srr.urdf (robot description, URDF)
Before this commit: robot srr, 14 links, 13 joints
Links:
- link Front_Left: geometry collision mesh filename=package://srr_sim/meshes/srr/Front_Left.STL; visual mesh filename=package://srr_sim/meshes/srr/Front_Left.STL
- link Front_Left_Rev_Link: geometry collision mesh filename=package://srr_sim/meshes/srr/Front_Left_Rev_Link.STL; visual mesh filename=package://srr_sim/meshes/srr/Front_Left_Rev_Link.STL
- link Front_Left_Wheel: geometry collision mesh filename=package://srr_sim/meshes/srr/Front_Left_Wheel.STL; visual mesh filename=package://srr_sim/meshes/srr/Front_Left_Wheel.STL
- link Front_Right: geometry collision mesh filename=package://srr_sim/meshes/srr/Front_Right.STL; visual mesh filename=package://srr_sim/meshes/srr/Front_Right.STL
- link Front_Right_Rev_Link: geometry collision mesh filename=package://srr_sim/meshes/srr/Front_Right_Rev_Link.STL; visual mesh filename=package://srr_sim/meshes/srr/Front_Right_Rev_Link.STL
- link Front_Right_Wheel: geometry collision mesh filename=package://srr_sim/meshes/srr/Front_Right_Wheel.STL; visual mesh filename=package://srr_sim/meshes/srr/Front_Right_Wheel.STL
- link Rear_Left: geometry collision mesh filename=package://srr_sim/meshes/srr/Rear_Left.STL; visual mesh filename=package://srr_sim/meshes/srr/Rear_Left.STL
- link Rear_Left_Fixed_Link: geometry collision mesh filename=package://srr_sim/meshes/srr/Rear_Left_Fixed_Link.STL; visual mesh filename=package://srr_sim/meshes/srr/Rear_Left_Fixed_Link.STL
- link Rear_Left_Wheel: geometry collision mesh filename=package://srr_sim/meshes/srr/Rear_Left_Wheel.STL; visual mesh filename=package://srr_sim/meshes/srr/Rear_Left_Wheel.STL
- link Rear_Right: geometry collision mesh filename=package://srr_sim/meshes/srr/Rear_Right.STL; visual mesh filename=package://srr_sim/meshes/srr/Rear_Right.STL
- link Rear_Right_Fixed_Link: geometry collision mesh filename=package://srr_sim/meshes/srr/Rear_Right_Fixed_Link.STL; visual mesh filename=package://srr_sim/meshes/srr/Rear_Right_Fixed_Link.STL
- link Rear_Right_Wheel: geometry collision mesh filename=package://srr_sim/meshes/srr/Rear_Right_Wheel.STL; visual mesh filename=package://srr_sim/meshes/srr/Rear_Right_Wheel.STL
- link base_link: geometry collision mesh filename=package://srr_sim/meshes/srr/base_link.STL; visual mesh filename=package://srr_sim/meshes/srr/base_link.STL

Commit message: Added proper joint limits to the vehicle's legs.

File: src/srr_sim/urdf/srr.urdf (robot description, URDF)
Before this commit: robot srr, 14 links, 13 joints
Joints:
- joint FL_Joint: limit lower=-1.5707963 upper=1.5707963 effort=125 velocity=0 -> lower=-0.767945 upper=0.0 effort=125 velocity=0
- joint FR_Joint: limit lower=-1.5707963 upper=1.5707963 effort=125 velocity=0 -> lower=-0.767945 upper=0.0 effort=125 velocity=0
- joint RL_Joint: limit lower=-1.5707963 upper=1.5707963 effort=125 velocity=0 -> lower=0.0 upper=0.767945 effort=125 velocity=0
- joint RR_Joint: limit lower=-1.5707963 upper=1.5707963 effort=125 velocity=0 -> lower=0.0 upper=0.767945 effort=125 velocity=0

Commit message: Finished contact angle estimation for first wheel

File: src/srr_sim/urdf/srr.urdf (robot description, URDF)
Before this commit: robot srr, 14 links, 13 joints
Joints:
- joint FL_Rev_Joint: limit lower=-0.218166 upper=0.218166 effort=125 velocity=0 -> lower=-0.02 upper=0.02 effort=125 velocity=0
- joint FL_Wheel_Joint: origin xyz=0 -0.06096 0 rpy=0 0 -1.2844 -> xyz=0 -0.06096 0 rpy=0 0 0
- joint FR_Rev_Joint: limit lower=-0.218166 upper=0.218166 effort=125 velocity=0 -> lower=-0.02 upper=0.02 effort=125 velocity=0
- joint FR_Wheel_Joint: origin xyz=0 -0.06096 0 rpy=0 0 -1.2319 -> xyz=0 -0.06096 0 rpy=0 0 0
- joint RL_Wheel_Joint: origin xyz=0 -0.04445 0 rpy=0 0 0.62124 -> xyz=0 -0.04445 0 rpy=0 0 0
- joint RR_Wheel_Joint: origin xyz=0 -0.04445 0 rpy=0 0 3.0007 -> xyz=0 -0.04445 0 rpy=0 0 0
