Commit message: WHITE-SPACE: no functional changes, just reorganizing/cleaning XML-like code and whitespace.

File: src/srr_sim/urdf/srr_integrated.urdf.xacro (robot description, xacro)
@@ -3,4 +3,31 @@
   <xacro:include filename="srr.urdf"/>
   <!-- ROBOT JOINT TRANSMISSIONS -->
+  <transmission name="FL_Transmitter">
+    <type>transmission_interface/SimpleTransmission</type>
+    <joint name="FL_Joint">
+      <hardwareInterface>hardware_interface/EffortJointInterface</hardwareInterface>
+    </joint>
+    <actuator name="FL_Motor">
+      <mechanicalReduction>50</mechanicalReduction>
+    </actuator>
+  </transmission>
+  <transmission name="FL_Wheel_Transmitter">
+    <type>transmission_interface/SimpleTransmission</type>
+    <joint name="FL_Wheel_Joint">
+      <hardwareInterface>hardware_interface/EffortJointInterface</hardwareInterface>
+    </joint>
+    <actuator name="FL_Wheel_Motor">
+      <mechanicalReduction>50</mechanicalReduction>
+    </actuator>
+  </transmission>
+  <transmission name="FR_Wheel_Transmitter">
+    <type>transmission_interface/SimpleTransmission</type>
+    <joint name="FR_Wheel_Joint">
+      <hardwareInterface>hardware_interface/EffortJointInterface</hardwareInterface>
+    </joint>
+    <actuator name="FR_Wheel_Motor">
+      <mechanicalReduction>50</mechanicalReduction>
+    </actuator>
+  </transmission>
   <transmission name="FR_Transmitter">
     <type>transmission_interface/SimpleTransmission</type>
@@ -12,10 +39,19 @@
     </actuator>
   </transmission>
-  <transmission name="FL_Transmitter">
+  <transmission name="RL_Transmitter">
     <type>transmission_interface/SimpleTransmission</type>
-    <joint name="FL_Joint">
+    <joint name="RL_Joint">
       <hardwareInterface>hardware_interface/EffortJointInterface</hardwareInterface>
     </joint>
-    <actuator name="FL_Motor">
+    <actuator name="RL_Motor">
+      <mechanicalReduction>50</mechanicalReduction>
+    </actuator>
+  </transmission>
+  <transmission name="RL_Wheel_Transmitter">
+    <type>transmission_interface/SimpleTransmission</type>
+    <joint name="RL_Wheel_Joint">
+      <hardwareInterface>hardware_interface/EffortJointInterface</hardwareInterface>
+    </joint>
+    <actuator name="RL_Wheel_Motor">
       <mechanicalReduction>50</mechanicalReduction>
     </actuator>
@@ -30,31 +66,4 @@
     </actuator>
   </transmission>
-  <transmission name="RL_Transmitter">
-    <type>transmission_interface/SimpleTransmission</type>
-    <joint name="RL_Joint">
-      <hardwareInterface>hardware_interface/EffortJointInterface</hardwareInterface>
-    </joint>
-    <actuator name="RL_Motor">
-      <mechanicalReduction>50</mechanicalReduction>
-    </actuator>
-  </transmission>
-  <transmission name="FR_Wheel_Transmitter">
-    <type>transmission_interface/SimpleTransmission</type>
-    <joint name="FR_Wheel_Joint">
-      <hardwareInterface>hardware_interface/EffortJointInterface</hardwareInterface>
-    </joint>
-    <actuator name="FR_Wheel_Motor">
-      <mechanicalReduction>50</mechanicalReduction>
-    </actuator>
-  </transmission>
-  <transmission name="FL_Wheel_Transmitter">
-    <type>transmission_interface/SimpleTransmission</type>
-    <joint name="FL_Wheel_Joint">
-      <hardwareInterface>hardware_interface/EffortJointInterface</hardwareInterface>
-    </joint>
-    <actuator name="FL_Wheel_Motor">
-      <mechanicalReduction>50</mechanicalReduction>
-    </actuator>
-  </transmission>
   <transmission name="RR_Wheel_Transmitter">
     <type>transmission_interface/SimpleTransmission</type>
@@ -63,13 +72,4 @@
     </joint>
     <actuator name="RR_Wheel_Motor">
-      <mechanicalReduction>50</mechanicalReduction>
-    </actuator>
-  </transmission>
-  <transmission name="RL_Wheel_Transmitter">
-    <type>transmission_interface/SimpleTransmission</type>
-    <joint name="RL_Wheel_Joint">
-      <hardwareInterface>hardware_interface/EffortJointInterface</hardwareInterface>
-    </joint>
-    <actuator name="RL_Wheel_Motor">
       <mechanicalReduction>50</mechanicalReduction>
     </actuator>

Commit message: Quickly added initial IMU sensor to vehicle chassis.

File: src/srr_sim/urdf/srr_integrated.urdf.xacro (robot description, xacro)
@@ -75,5 +75,5 @@
     </actuator>
   </transmission>
-  <!-- ROS CONTROL LIBRARY -->
+  <!-- GAZEBO PLUGINS/LIBRARIES -->
   <gazebo>
     <plugin name="gazebo_ros_control" filename="libgazebo_ros_control.so">
@@ -82,4 +82,43 @@
       <legacyModeNS>true</legacyModeNS>
     </plugin>
+    <plugin name="imu_control" filename="libgazebo_ros_imu.so">
+      <alwaysOn>true</alwaysOn>
+      <updateRate>50</updateRate>
+      <bodyName>IMU_Link</bodyName>
+      <topicName>/srr_integrated/imu_data</topicName>
+      <serviceName>/srr_integrated/imu_data_service</serviceName>
+      <gaussianNoise>1e-08</gaussianNoise>
+    </plugin>
   </gazebo>
+  <!-- IMU -->
+  <joint name="IMU_Joint" type="fixed">
+    <origin xyz="0 0 0" rpy="0 0 0"/>
+    <parent link="Vehicle_Base_Link"/>
+    <child link="IMU_Link"/>
+  </joint>
+  <link name="IMU_Link">
+    <inertial>
+      <mass value="0.001"/>
+      <origin rpy="0 0 0" xyz="0 0 0"/>
+      <inertia
+        ixx="0.0001"
+        ixy="0"
+        ixz="0"
+        iyy="0.000001"
+        iyz="0"
+        izz="0.0001"/>
+    </inertial>
+    <visual>
+      <origin rpy="0 0 0" xyz="0 0 0"/>
+      <geometry>
+        <box size="0.001 0.001 0.001"/>
+      </geometry>
+    </visual>
+    <collision>
+      <origin rpy="0 0 0" xyz="0 0 0"/>
+      <geometry>
+        <box size="0.001 0.001 0.001"/>
+      </geometry>
+    </collision>
+  </link>
 </robot>

Commit message: Add basic controllers for the front steerable wheels

File: src/srr_sim/urdf/srr_integrated.urdf.xacro (robot description, xacro)
@@ -9,4 +9,13 @@
     </joint>
     <actuator name="FL_Motor">
+      <mechanicalReduction>50</mechanicalReduction>
+    </actuator>
+  </transmission>
+  <transmission name="FL_Rev_Transmitter">
+    <type>transmission_interface/SimpleTransmission</type>
+    <joint name="FL_Rev_Joint">
+      <hardwareInterface>hardware_interface/EffortJointInterface</hardwareInterface>
+    </joint>
+    <actuator name="FL_Rev_Motor">
       <mechanicalReduction>50</mechanicalReduction>
     </actuator>
@@ -27,4 +36,13 @@
     </joint>
     <actuator name="FR_Wheel_Motor">
+      <mechanicalReduction>50</mechanicalReduction>
+    </actuator>
+  </transmission>
+  <transmission name="FR_Rev_Transmitter">
+    <type>transmission_interface/SimpleTransmission</type>
+    <joint name="FR_Rev_Joint">
+      <hardwareInterface>hardware_interface/EffortJointInterface</hardwareInterface>
+    </joint>
+    <actuator name="FR_Rev_Motor">
       <mechanicalReduction>50</mechanicalReduction>
     </actuator>
