Commit message: Added combined launch config, for the sra mounted onto the srr
To keep the environment as clean as possible, some launch, URDF/XACRO,
STL, ROS node, etc. files were modified / cleaned up in an effort to
maintain consistency and uniqueness when necessary across all files
and launch configurations. Also added some instructions to the README
to use each config.

File: src/srr_sim/urdf/sra.urdf (robot description, URDF)
Before this commit: robot sra, 8 links, 7 joints
Links:
- removed link base_link
- added link ArmBaseLink, mass 0.08044; collision mesh filename=package://srr_sim/meshes/sra/ArmBaseLink.STL; visual mesh filename=package://srr_sim/meshes/sra/ArmBaseLink.STL
- added link ArmDummyLink
Joints:
- added joint ArmDummyJoint: type fixed, parent ArmDummyLink, child ArmBaseLink, origin xyz=0 0 0 rpy=0 0 0
- joint BaseJoint: parent base_link -> ArmBaseLink

File: src/srr_sim/urdf/sra_integrated.urdf.xacro (robot description, xacro)
@@ -3,8 +3,8 @@
   <!-- WORLD -->
   <link name="world"/>
-  <joint name="WorldJoint" type="fixed">
+  <joint name="ArmWorldJoint" type="fixed">
     <origin rpy="0 0 0" xyz="0 0 0"/>
     <parent link="world"/>
-    <child link="base_link"/>
+    <child link="ArmDummyLink"/>
   </joint>
   <!-- ROBOT -->

File: src/srr_sim/urdf/srr.urdf (robot description, URDF)
Before this commit: robot srr, 14 links, 13 joints
Links:
- removed link base_link
- removed link dummy_link
- added link VehicleDummyLink
- added link Vehicle_Base_Link, mass 16.6873668690236; collision mesh filename=package://srr_sim/meshes/srr/Vehicle_Base_Link.STL; visual mesh filename=package://srr_sim/meshes/srr/Vehicle_Base_Link.STL
Joints:
- removed joint DummyJoint
- added joint VehicleDummyJoint: type fixed, parent VehicleDummyLink, child Vehicle_Base_Link, origin xyz=0 0 0 rpy=0 0 0
- joint FL_Joint: parent base_link -> Vehicle_Base_Link
- joint FR_Joint: parent base_link -> Vehicle_Base_Link
- joint RL_Joint: parent base_link -> Vehicle_Base_Link
- joint RR_Joint: parent base_link -> Vehicle_Base_Link

Commit message: Added basic/dummy arm controllers and arm teleop script

File: src/srr_sim/urdf/sra.urdf (robot description, URDF)
Before this commit: robot sra, 9 links, 8 joints
Joints:
- joint BaseJoint: limit lower=-3.14159265 upper=3.14159265 effort=0 velocity=0 -> lower=-3.14159265 upper=3.14159265 effort=125 velocity=0
- joint ElbowJoint: limit lower=-3.14159265 upper=3.14159265 effort=0 velocity=0 -> lower=-3.14159265 upper=3.14159265 effort=125 velocity=0
- joint ShoulderJoint: limit lower=-3.14159265 upper=3.14159265 effort=0 velocity=0 -> lower=-3.14159265 upper=3.14159265 effort=125 velocity=0
- joint WristJoint: limit lower=-3.14159265 upper=3.14159265 effort=0 velocity=0 -> lower=-3.14159265 upper=3.14159265 effort=125 velocity=0

File: src/srr_sim/urdf/sra_integrated.urdf.xacro (robot description, xacro)
@@ -10,4 +10,41 @@
   <!-- ROBOT -->
   <xacro:include filename="sra.urdf"/>
+  <!-- ROBOT JOINT TRANSMISSIONS -->
+  <transmission name="BaseJoint_Transmitter">
+    <type>transmission_interface/SimpleTransmission</type>
+    <joint name="BaseJoint">
+      <hardwareInterface>hardware_interface/EffortJointInterface</hardwareInterface>
+    </joint>
+    <actuator name="BaseJoint_Motor">
+      <mechanicalReduction>50</mechanicalReduction>
+    </actuator>
+  </transmission>
+  <transmission name="ShoulderJoint_Transmitter">
+    <type>transmission_interface/SimpleTransmission</type>
+    <joint name="ShoulderJoint">
+      <hardwareInterface>hardware_interface/EffortJointInterface</hardwareInterface>
+    </joint>
+    <actuator name="ShoulderJoint_Motor">
+      <mechanicalReduction>50</mechanicalReduction>
+    </actuator>
+  </transmission>
+  <transmission name="ElbowJoint_Transmitter">
+    <type>transmission_interface/SimpleTransmission</type>
+    <joint name="ElbowJoint">
+      <hardwareInterface>hardware_interface/EffortJointInterface</hardwareInterface>
+    </joint>
+    <actuator name="ElbowJoint_Motor">
+      <mechanicalReduction>50</mechanicalReduction>
+    </actuator>
+  </transmission>
+  <transmission name="WristJoint">
+    <type>transmission_interface/SimpleTransmission</type>
+    <joint name="WristJoint">
+      <hardwareInterface>hardware_interface/EffortJointInterface</hardwareInterface>
+    </joint>
+    <actuator name="WristJoint_Motor">
+      <mechanicalReduction>50</mechanicalReduction>
+    </actuator>
+  </transmission>
   <!-- ROS CONTROL LIBRARY -->
   <gazebo>

Commit message: Added the arm urdf and meshes

File: src/srr_sim/urdf/sra.urdf (robot description, URDF)
Before this commit: robot sra, 9 links, 8 joints
Links:
- removed link Gripper
- added link GripperToFinger, mass 0.064061; collision mesh filename=package://srr_sim/meshes/sra/GripperToFinger.STL; visual mesh filename=package://srr_sim/meshes/sra/GripperToFinger.STL
- added link LeftFinger, mass 0.000346143112791696; collision mesh filename=package://srr_sim/meshes/sra/LeftFinger.STL; visual mesh filename=package://srr_sim/meshes/sra/LeftFinger.STL
- added link RightFinger, mass 0.00034614; collision mesh filename=package://srr_sim/meshes/sra/RightFinger.STL; visual mesh filename=package://srr_sim/meshes/sra/RightFinger.STL
- link BaseToShoulderLink: mass 0.0540161279717926 -> 0.06206
- link ElbowDummyToElbowLink: mass 0.0573187162898318 -> 0.057319
- link ElbowToWristDummyLink: mass 0.254788454624903 -> 0.254411955196347
- link ShoulderToElbowDummyLink: mass 0.214557043401322 -> 0.20651
- link WristDummyToWristLink: mass 0.0181588599237565 -> 0.018159
- link WristToGripperLink: mass 0.064171 -> 0.0640611944357688
Joints:
- added joint LFingerJoint: type revolute, parent GripperToFinger, child LeftFinger, origin xyz=-0.00762 0.009525 0.001905 rpy=1.5708 0.88304 0, axis 0 0 1, limit lower=-3.14159265 upper=3.14159265 effort=125 velocity=0
- added joint RFingerJoint: type revolute, parent GripperToFinger, child RightFinger, origin xyz=0.00762 0.009525 0.001905 rpy=1.5708 0.98268 -3.14159265, axis 0 0 1, limit lower=-3.14159265 upper=3.14159265 effort=125 velocity=0
- joint BaseJoint: axis 0 1 0 -> 0 0 1; origin xyz=0 0 0.0254 rpy=1.5708 0 1.4018 -> xyz=0 0 0.073354 rpy=0 0 0
- joint ElbowDummyJoint: origin xyz=0.12391 0.12273 0 rpy=3.1416 1.5699 2.3621 -> xyz=0 -0.19622 0 rpy=-1.5699 0 -1.5708
- joint ElbowJoint: origin xyz=0 0.020955 0.044653 rpy=-1.5708 -0.78332 1.5708 -> xyz=0 0.000127 0.044653 rpy=1.5708 0 0
- joint GripperJoint: axis 0 0 1 -> 0 0 0; child Gripper -> GripperToFinger; limit lower=-3.14159265 upper=3.14159265 effort=0 velocity=0 -> (none); origin xyz=-0.027305 -0.00762 0 rpy=0 0 0.65153 -> xyz=0 0.0254 0.009525 rpy=-1.5708 0 0; type revolute -> fixed
- joint ShoulderJoint: origin xyz=0 0.05 0 rpy=0 0 -0.35492 -> xyz=0 0 0 rpy=-1.5708 0 0
- joint WristDummyJoint: origin xyz=0.20384 0 0 rpy=1.5708 -1.537 -1.5708 -> xyz=0.2267 0 0 rpy=0.033844 0 0.00012806
- joint WristJoint: origin xyz=0 0 -0.02286 rpy=-1.5708 -0.36389 1.5708 -> xyz=0 0 0 rpy=0 0 -1.5708
